File: pcbs/src/mcu_adapter.kicad_pcb (KiCad board)
At the start: 2 copper layers, 30 x 21 mm, 5 parts, among them U1 XIAO-THRUHOLE

Commit message: re added missing kicad files
Parts:
- U$1, U$2: footprint CONN3X2_NRPN032PAEN-RC_vf.TnALXNQpQbKa17UGSM3jDw -> mcu_adapter:CONN3X2_NRPN032PAEN-RC_vf.TnALXNQpQbKa17UGSM3jDw
- U1: footprint XIAO-GENERIC-THRUHOLE-MODULE14P-2.54-21X17.8MM_vf.79dh4xraRyqeNIxPyZlsGg -> mcu_adapter:XIAO-GENERIC-THRUHOLE-MODULE14P-2.54-21X17.8MM_vf.79dh4xraRyqeNIxPyZlsGg
- UNK_HOLE_0: footprint dummyfp0 -> mcu_adapter:dummyfp0
- UNK_HOLE_1: footprint dummyfp1 -> mcu_adapter:dummyfp1
